Commit message: add LIDAR sensor and integrate RViz2 visualization

File: src/hexarover_description/urdf/hexarover.urdf.xacro (robot description, xacro)
@@ -1,101 +1,123 @@
 <?xml version="1.0"?>
 <robot name="hexarover" xmlns:xacro="http://www.ros.org/wiki/xacro">
+  <material name="silver">
+    <color rgba="0.8 0.8 0.8 1"/>
+  </material>
+  <material name="black">
+    <color rgba="0.1 0.1 0.1 1"/>
+  </material>
+  <material name="red">
+    <color rgba="1 0 0 1"/>
+  </material>
   <link name="base_link">
     <visual>
+      <origin xyz="0 0 0.04" rpy="0 0 0"/> <geometry>
+        <box size="0.45 0.16 0.08"/> </geometry>
+      <material name="silver"/>
+    </visual>
+    <collision>
+      <origin xyz="0 0 0.04" rpy="0 0 0"/>
       <geometry>
-        <box size="0.6 0.4 0.15"/>
+        <box size="0.45 0.16 0.08"/>
       </geometry>
-      <material name="orange">
-        <color rgba="1 0.5 0 1"/>
-      </material>
+    </collision>
+    <inertial>
+      <mass value="5.0"/>
+      <inertia ixx="0.04" ixy="0" ixz="0" iyy="0.1" iyz="0" izz="0.1"/>
+    </inertial>
+  </link>
+  <xacro:macro name="wheel" params="prefix side x_pos y_pos friction">
+    <link name="${prefix}_${side}_wheel">
+      <visual>
+        <geometry>
+          <cylinder radius="0.065" length="0.07"/> </geometry>
+        <material name="black"/>
+      </visual>
+      <collision>
+        <geometry>
+          <cylinder radius="0.065" length="0.07"/>
+        </geometry>
+      </collision>
+      <inertial>
+        <mass value="0.8"/>
+        <inertia ixx="0.001" ixy="0" ixz="0" iyy="0.001" iyz="0" izz="0.001"/>
+      </inertial>
+    </link>
+    <joint name="${prefix}_${side}_wheel_joint" type="continuous">
+      <parent link="base_link"/>
+      <child link="${prefix}_${side}_wheel"/>
+      <origin xyz="${x_pos} ${y_pos} 0" rpy="-1.5707 0 0"/>
+      <axis xyz="0 0 1"/>
+    </joint>
+    <gazebo reference="${prefix}_${side}_wheel">
+      <mu1>${friction}</mu1> <mu2>${friction}</mu2> <material>Gazebo/Black</material>
+    </gazebo>
+  </xacro:macro>
+  <xacro:wheel prefix="mid" side="left"  x_pos="0"     y_pos="0.13" friction="1.0"/>
+  <xacro:wheel prefix="mid" side="right" x_pos="0"     y_pos="-0.13" friction="1.0"/>
+  <xacro:wheel prefix="front" side="left"  x_pos="0.16"  y_pos="0.13" friction="0.2"/>
+  <xacro:wheel prefix="front" side="right" x_pos="0.16"  y_pos="-0.13" friction="0.2"/>
+  <xacro:wheel prefix="rear" side="left"  x_pos="-0.16" y_pos="0.13" friction="0.2"/>
+  <xacro:wheel prefix="rear" side="right" x_pos="-0.16" y_pos="-0.13" friction="0.2"/>
+  <link name="lidar_link">
+    <visual>
+      <geometry>
+        <cylinder radius="0.035" length="0.04"/>
+      </geometry>
+      <material name="red"/>
     </visual>
     <collision>
       <geometry>
-        <box size="0.6 0.4 0.15"/>
+        <cylinder radius="0.035" length="0.04"/>
       </geometry>
     </collision>
     <inertial>
-      <mass value="10.0"/>
-      <inertia ixx="0.1" ixy="0" ixz="0" iyy="0.1" iyz="0" izz="0.1"/>
+      <mass value="0.1"/>
+      <inertia ixx="0.0001" ixy="0" ixz="0" iyy="0.0001" iyz="0" izz="0.0001"/>
     </inertial>
   </link>
-  <link name="left_wheel">
-    <visual>
-      <geometry>
-        <cylinder radius="0.12" length="0.08"/>
-      </geometry>
-      <material name="black">
-        <color rgba="0 0 0 1"/>
-      </material>
-    </visual>
-    <collision>
-      <geometry>
-        <cylinder radius="0.12" length="0.08"/>
-      </geometry>
-    </collision>
-    <inertial>
-      <mass value="2.0"/>
-      <inertia ixx="0.01" ixy="0" ixz="0" iyy="0.01" iyz="0" izz="0.01"/>
-    </inertial>
-  </link>
-  <joint name="left_wheel_joint" type="continuous">
+  <joint name="lidar_joint" type="fixed">
     <parent link="base_link"/>
-    <child link="left_wheel"/>
-    <origin xyz="0 0.24 0" rpy="-1.5707 0 0"/>
-    <axis xyz="0 0 1"/>
-  </joint>
-  <link name="right_wheel">
-    <visual>
-      <geometry>
-        <cylinder radius="0.12" length="0.08"/>
-      </geometry>
-      <material name="black"/>
-    </visual>
-    <collision>
-      <geometry>
-        <cylinder radius="0.12" length="0.08"/>
-      </geometry>
-    </collision>
-    <inertial>
-      <mass value="2.0"/>
-      <inertia ixx="0.01" ixy="0" ixz="0" iyy="0.01" iyz="0" izz="0.01"/>
-    </inertial>
-  </link>
-  <joint name="right_wheel_joint" type="continuous">
-    <parent link="base_link"/>
-    <child link="right_wheel"/>
-    <origin xyz="0 -0.24 0" rpy="-1.5707 0 0"/>
-    <axis xyz="0 0 1"/>
-  </joint>
-  <link name="caster_wheel">
-    <visual>
-      <geometry>
-        <sphere radius="0.06"/>
-      </geometry>
-      <material name="grey"/>
-    </visual>
-    <collision>
-      <geometry>
-        <sphere radius="0.06"/>
-      </geometry>
-    </collision>
-    <inertial>
-      <mass value="0.5"/>
-      <inertia ixx="0.001" ixy="0" ixz="0" iyy="0.001" iyz="0" izz="0.001"/>
-    </inertial>
-  </link>
-  <joint name="caster_joint" type="fixed">
-    <parent link="base_link"/>
-    <child link="caster_wheel"/>
-    <origin xyz="0.25 0 -0.06"/>
+    <child link="lidar_link"/>
+    <origin xyz="0.05 0 0.10" rpy="0 0 0"/>
   </joint>
   <gazebo>
     <plugin filename="gz-sim-diff-drive-system" name="gz::sim::systems::DiffDrive">
-      <left_joint>left_wheel_joint</left_joint>
-      <right_joint>right_wheel_joint</right_joint>
-      <wheel_separation>0.48</wheel_separation>
-      <wheel_radius>0.12</wheel_radius>
+      <left_joint>mid_left_wheel_joint</left_joint>
+      <right_joint>mid_right_wheel_joint</right_joint>
+      <wheel_separation>0.26</wheel_separation>
+      <wheel_radius>0.065</wheel_radius>
       <topic>cmd_vel</topic>
+      <max_linear_acceleration>2.0</max_linear_acceleration>
+    </plugin>
+    <plugin filename="gz-sim-sensors-system" name="gz::sim::systems::Sensors">
+      <render_engine>ogre2</render_engine>
+    </plugin>
+    <plugin filename="gz-sim-joint-state-publisher-system" name="gz::sim::systems::JointStatePublisher">
+      <topic>joint_states</topic> <update_rate>30</update_rate>
     </plugin>
   </gazebo>
+  <gazebo reference="lidar_link">
+    <sensor name="lidar" type="gpu_lidar">
+      <pose>0 0 0 0 0 0</pose>
+      <always_on>true</always_on>
+      <visualize>true</visualize>
+      <update_rate>10</update_rate>
+      <ray>
+        <scan>
+          <horizontal>
+            <samples>360</samples>
+            <resolution>1</resolution>
+            <min_angle>-3.14</min_angle>
+            <max_angle>3.14</max_angle>
+          </horizontal>
+        </scan>
+        <range>
+          <min>0.15</min> <max>10.0</max>
+        </range>
+      </ray>
+      <topic>scan</topic>
+      <gz_frame_id>lidar_link</gz_frame_id>
+    </sensor>
+  </gazebo>
 </robot>

Commit message: Dodanie IMU i SLAM

File: src/hexarover_description/urdf/hexarover.urdf.xacro (robot description, xacro)
@@ -10,4 +10,7 @@
     <color rgba="1 0 0 1"/>
   </material>
+  <material name="green">
+  <color rgba="0 1 0 1"/>
+</material>
   <link name="base_link">
     <visual>
@@ -82,4 +85,26 @@
     <origin xyz="0.05 0 0.10" rpy="0 0 0"/>
   </joint>
+  <link name="imu_link">
+    <visual>
+      <geometry>
+         <cylinder radius="0.035" length="0.04"/>
+       </geometry>
+      <material name="green"/>
+    </visual>
+        <collision>
+      <geometry>
+        <cylinder radius="0.035" length="0.02"/>
+      </geometry>
+    </collision>
+    <inertial>
+      <mass value="0.01"/>
+      <inertia ixx="0.00001" ixy="0" ixz="0" iyy="0.00001" iyz="0" izz="0.00001"/>
+    </inertial>
+  </link>
+  <joint name="imu_joint" type="fixed">
+    <parent link="base_link"/>
+    <child link="imu_link"/>
+    <origin xyz="0.2 0 0.10" rpy="0 0 0"/>
+    </joint>
   <gazebo>
     <plugin filename="gz-sim-diff-drive-system" name="gz::sim::systems::DiffDrive">
@@ -90,4 +115,9 @@
       <topic>cmd_vel</topic>
       <max_linear_acceleration>2.0</max_linear_acceleration>
+      <odom_publish_frequency>0</odom_publish_frequency>
+      <publish_odom>false</publish_odom>
+      <publish_odom_tf>false</publish_odom_tf>
+      <child_frame_id>base_link</child_frame_id>
+      <odom_topic>odometry_off</odom_topic>
     </plugin>
     <plugin filename="gz-sim-sensors-system" name="gz::sim::systems::Sensors">
@@ -96,4 +126,6 @@
     <plugin filename="gz-sim-joint-state-publisher-system" name="gz::sim::systems::JointStatePublisher">
       <topic>joint_states</topic> <update_rate>30</update_rate>
+    </plugin>
+    <plugin filename="gz-sim-imu-system" name="gz::sim::systems::Imu">
     </plugin>
   </gazebo>
@@ -121,3 +153,55 @@
     </sensor>
   </gazebo>
+  <gazebo reference="imu_link">
+    <sensor name="imu_sensor" type="imu">
+      <pose>0 0 0 0 0 0</pose>
+      <always_on>true</always_on>
+      <visualize>true</visualize>
+      <update_rate>10</update_rate>
+      <imu>
+        <angular_velocity>
+          <x>
+            <noise type="gaussian">
+              <mean>0.0</mean>
+              <stddev>0.0</stddev>
+            </noise>
+          </x>
+          <y>
+            <noise type="gaussian">
+              <mean>0.0</mean>
+              <stddev>0.0</stddev>
+            </noise>
+          </y>
+          <z>
+            <noise type="gaussian">
+              <mean>0.0</mean>
+              <stddev>0.0</stddev>
+            </noise>
+          </z>
+        </angular_velocity>
+        <linear_acceleration>
+          <x>
+            <noise type="gaussian">
+              <mean>0.0</mean>
+              <stddev>0.0</stddev>
+            </noise>
+          </x>
+          <y>
+            <noise type="gaussian">
+              <mean>0.0</mean>
+              <stddev>0.0</stddev>
+            </noise>
+          </y>
+          <z>
+            <noise type="gaussian">
+              <mean>0.0</mean>
+              <stddev>0.0</stddev>
+            </noise>
+          </z>
+        </linear_acceleration>
+      </imu>
+      <topic>/imu</topic>
+      <gz_frame_id>imu_link</gz_frame_id>
+      </sensor>
+  </gazebo>
 </robot>

Commit message: not working nav2

File: src/hexarover_description/urdf/hexarover.urdf.xacro (robot description, xacro)
@@ -12,5 +12,5 @@
   <material name="green">
   <color rgba="0 1 0 1"/>
-</material>
+  </material>
   <link name="base_link">
     <visual>

Commit message: adding camera, human to sim world & rqt_image_view

File: src/hexarover_description/urdf/hexarover.urdf.xacro (robot description, xacro)
@@ -107,4 +107,33 @@
     <origin xyz="0.2 0 0.10" rpy="0 0 0"/>
     </joint>
+    <link name="camera_link">
+    <visual>
+      <geometry>
+        <box size="0.02 0.05 0.03"/>
+      </geometry>
+      <material name="black"/>
+    </visual>
+    <collision>
+      <geometry>
+        <box size="0.02 0.05 0.03"/>
+      </geometry>
+    </collision>
+    <inertial>
+      <mass value="0.05"/>
+      <inertia ixx="0.00001" ixy="0" ixz="0" iyy="0.00001" iyz="0" izz="0.00001"/>
+    </inertial>
+  </link>
+  <joint name="camera_joint" type="fixed">
+    <parent link="base_link"/>
+    <child link="camera_link"/>
+    <origin xyz="0.22 0 0.18" rpy="0 0 0"/>
+  </joint>
+  <link name="camera_link_optical"></link>
+  <joint name="camera_optical_joint" type="fixed">
+    <parent link="camera_link"/>
+    <child link="camera_link_optical"/>
+    <!-- Standardowa konwersja osi optycznych OpenCV -->
+    <origin xyz="0 0 0" rpy="-1.57079632679 0 -1.57079632679"/>
+  </joint>
   <gazebo>
     <plugin filename="gz-sim-diff-drive-system" name="gz::sim::systems::DiffDrive">
@@ -205,3 +234,30 @@
       </sensor>
   </gazebo>
+  <gazebo reference="camera_link">
+    <sensor name="camera_sensor" type="camera">
+      <pose>0 0 0 0 0 0</pose>
+      <always_on>true</always_on>
+      <visualize>true</visualize>
+      <update_rate>30.0</update_rate>
+      <camera name="hexarover_camera">
+        <horizontal_fov>1.047</horizontal_fov>
+        <image>
+          <width>800</width>
+          <height>600</height>
+          <format>R8G8B8</format>
+        </image>
+        <clip>
+          <near>0.02</near>
+          <far>100.0</far>
+        </clip>
+        <noise>
+          <type>gaussian</type>
+          <mean>0.0</mean>
+          <stddev>0.007</stddev>
+        </noise>
+      </camera>
+      <topic>/image_raw</topic>
+      <gz_frame_id>camera_link_optical</gz_frame_id>
+    </sensor>
+  </gazebo>
 </robot>

Commit message: adding sensor fusin human pos estimation and its rivizz vizualiztion

File: src/hexarover_description/urdf/hexarover.urdf.xacro (robot description, xacro)
@@ -127,5 +127,5 @@
     <parent link="base_link"/>
     <child link="camera_link"/>
-    <origin xyz="0.22 0 0.18" rpy="0 0 0"/>
+    <origin xyz="0.22 0 0.18" rpy="0 -0.26 0"/>
   </joint>
   <link name="camera_link_optical"></link>
@@ -241,5 +241,5 @@
       <update_rate>30.0</update_rate>
       <camera name="hexarover_camera">
-        <horizontal_fov>1.047</horizontal_fov>
+        <horizontal_fov>1.344</horizontal_fov>
         <image>
           <width>800</width>

Commit message: adding sonar to robot model, sonar topics and glass obsticles + yolo script modified by marek

File: src/hexarover_description/urdf/hexarover.urdf.xacro (robot description, xacro)
@@ -11,6 +11,6 @@
   </material>
   <material name="green">
-  <color rgba="0 1 0 1"/>
-</material>
+    <color rgba="0 1 0 1"/>
+  </material>
   <link name="base_link">
     <visual>
@@ -106,6 +106,6 @@
     <child link="imu_link"/>
     <origin xyz="0.2 0 0.10" rpy="0 0 0"/>
-    </joint>
-    <link name="camera_link">
+  </joint>
+  <link name="camera_link">
     <visual>
       <geometry>
@@ -133,7 +133,60 @@
     <parent link="camera_link"/>
     <child link="camera_link_optical"/>
-    <!-- Standardowa konwersja osi optycznych OpenCV -->
     <origin xyz="0 0 0" rpy="-1.57079632679 0 -1.57079632679"/>
   </joint>
+  <!-- ======================== MAKRO DLA CZUJNIKÓW ULTRADŹWIĘKOWYCH ======================== -->
+  <xacro:macro name="sonar" params="name x y z yaw">
+    <link name="sonar_${name}_link">
+      <visual>
+        <geometry><box size="0.01 0.03 0.015"/></geometry>
+        <material name="black"/>
+      </visual>
+    </link>
+    <joint name="sonar_${name}_joint" type="fixed">
+      <parent link="base_link"/>
+      <child link="sonar_${name}_link"/>
+      <!-- Montaż używając zmiennych zdefiniowanych przy wywołaniu makra -->
+      <origin xyz="${x} ${y} ${z}" rpy="0 0 ${yaw}"/>
+    </joint>
+    <gazebo reference="sonar_${name}_link">
+      <sensor name="sonar_${name}_sensor" type="gpu_lidar">
+        <always_on>true</always_on>
+        <update_rate>10</update_rate>
+        <visualize>true</visualize>
+        <topic>/sonar_${name}</topic>
+        <ray>
+          <scan>
+            <horizontal>
+              <samples>10</samples>
+              <resolution>1</resolution>
+              <!-- Kąt widzenia sonaru: ok. 30 stopni (od -15 do +15) -->
+              <min_angle>-0.26</min_angle>
+              <max_angle>0.26</max_angle>
+            </horizontal>
+            <vertical>
+              <samples>5</samples>
+              <resolution>1</resolution>
+              <min_angle>-0.1</min_angle>
+              <max_angle>0.1</max_angle>
+            </vertical>
+          </scan>
+          <range>
+            <!-- Zasięg od 2cm do 4 metrów -->
+            <min>0.02</min>
+            <max>4.0</max>
+            <resolution>0.01</resolution>
+          </range>
+        </ray>
+        <gz_frame_id>sonar_${name}_link</gz_frame_id>
+      </sensor>
+    </gazebo>
+  </xacro:macro>
+  <!-- ======================== MONTAŻ 4 CZUJNIKÓW NA ROGACH ROBOTA ======================== -->
+  <!-- Przód: Leciutko skierowane na boki (kąty 0.4 rad = ~23 stopnie) -->
+  <xacro:sonar name="front_left"  x="0.22" y="0.08"  z="0.05" yaw="0.4"/>
+  <xacro:sonar name="front_right" x="0.22" y="-0.08" z="0.05" yaw="-0.4"/>
+  <!-- Tył: Skierowane mocniej na boki, by pokryć ślepe strefy (kąty 2.35 rad = ~135 stopni) -->
+  <xacro:sonar name="rear_left"   x="-0.22" y="0.08"  z="0.05" yaw="2.35"/>
+  <xacro:sonar name="rear_right"  x="-0.22" y="-0.08" z="0.05" yaw="-2.35"/>
   <gazebo>
     <plugin filename="gz-sim-diff-drive-system" name="gz::sim::systems::DiffDrive">
@@ -151,5 +204,5 @@
     </plugin>
     <plugin filename="gz-sim-sensors-system" name="gz::sim::systems::Sensors">
-      <render_engine>ogre2</render_engine>
+      <!-- render_engine puste zgodnie z Twoimi poprzednimi udanymi testami -->
     </plugin>
     <plugin filename="gz-sim-joint-state-publisher-system" name="gz::sim::systems::JointStatePublisher">
@@ -191,40 +244,22 @@
         <angular_velocity>
           <x>
-            <noise type="gaussian">
-              <mean>0.0</mean>
-              <stddev>0.0</stddev>
-            </noise>
+            <noise type="gaussian"><mean>0.0</mean><stddev>0.0</stddev></noise>
           </x>
           <y>
-            <noise type="gaussian">
-              <mean>0.0</mean>
-              <stddev>0.0</stddev>
-            </noise>
+            <noise type="gaussian"><mean>0.0</mean><stddev>0.0</stddev></noise>
           </y>
           <z>
-            <noise type="gaussian">
-              <mean>0.0</mean>
-              <stddev>0.0</stddev>
-            </noise>
+            <noise type="gaussian"><mean>0.0</mean><stddev>0.0</stddev></noise>
           </z>
         </angular_velocity>
         <linear_acceleration>
           <x>
-            <noise type="gaussian">
-              <mean>0.0</mean>
-              <stddev>0.0</stddev>
-            </noise>
+            <noise type="gaussian"><mean>0.0</mean><stddev>0.0</stddev></noise>
           </x>
           <y>
-            <noise type="gaussian">
-              <mean>0.0</mean>
-              <stddev>0.0</stddev>
-            </noise>
+            <noise type="gaussian"><mean>0.0</mean><stddev>0.0</stddev></noise>
           </y>
           <z>
-            <noise type="gaussian">
-              <mean>0.0</mean>
-              <stddev>0.0</stddev>
-            </noise>
+            <noise type="gaussian"><mean>0.0</mean><stddev>0.0</stddev></noise>
           </z>
         </linear_acceleration>
@@ -232,5 +267,5 @@
       <topic>/imu</topic>
       <gz_frame_id>imu_link</gz_frame_id>
-      </sensor>
+    </sensor>
   </gazebo>
   <gazebo reference="camera_link">
