Commit message: accurate model discription in gazebo version

File: src/hexarover_description/urdf/hexarover.urdf.xacro (robot description, xacro)
@@ -1,4 +1,26 @@
 <?xml version="1.0"?>
 <robot name="hexarover" xmlns:xacro="http://www.ros.org/wiki/xacro">
+  <!-- ================= WŁAŚCIWOŚCI (PROPERTIES) ================= -->
+  <!-- 1. WYMIARY GŁÓWNEJ BRYŁY (PODWOZIA) -->
+  <xacro:property name="chassis_length" value="0.38"/>
+  <xacro:property name="chassis_width"  value="0.12"/>
+  <xacro:property name="chassis_height" value="0.07"/>
+  <xacro:property name="chassis_z_offset" value="0.02"/>
+  <!-- 2. KOŁA -->
+  <xacro:property name="wheel_radius" value="0.0625"/>
+  <xacro:property name="wheel_length" value="0.06"/>
+  <xacro:property name="wheel_y_offset" value="0.12"/>
+  <xacro:property name="axle_x_offset" value="0.15"/>
+  <!-- 3. POZYCJA LIDARU -->
+  <xacro:property name="lidar_x" value="0.15"/>
+  <xacro:property name="lidar_y" value="0.00"/>
+  <xacro:property name="lidar_z" value="0.12"/>
+  <xacro:property name="lidar_yaw" value="0.0"/>
+  <!-- 4. POZYCJA IMU -->
+  <xacro:property name="imu_x" value="-0.15"/>
+  <xacro:property name="imu_y" value="0.00"/>
+  <xacro:property name="imu_z" value="0.06"/>
+  <xacro:property name="imu_yaw" value="0.0"/>
+  <!-- ========================================================== -->
   <material name="silver">
     <color rgba="0.8 0.8 0.8 1"/>
@@ -11,16 +33,19 @@
   </material>
   <material name="green">
-  <color rgba="0 1 0 1"/>
-  </material>
+    <color rgba="0 1 0 1"/>
+  </material>
+  <!-- BASE LINK -->
   <link name="base_link">
     <visual>
-      <origin xyz="0 0 0.04" rpy="0 0 0"/> <geometry>
-        <box size="0.45 0.16 0.08"/> </geometry>
+      <origin xyz="0 0 ${chassis_z_offset}" rpy="0 0 0"/>
+      <geometry>
+        <box size="${chassis_length} ${chassis_width} ${chassis_height}"/>
+      </geometry>
       <material name="silver"/>
     </visual>
     <collision>
-      <origin xyz="0 0 0.04" rpy="0 0 0"/>
-      <geometry>
-        <box size="0.45 0.16 0.08"/>
+      <origin xyz="0 0 ${chassis_z_offset}" rpy="0 0 0"/>
+      <geometry>
+        <box size="${chassis_length} ${chassis_width} ${chassis_height}"/>
       </geometry>
     </collision>
@@ -30,14 +55,16 @@
     </inertial>
   </link>
+  <!-- WHEEL MACRO -->
   <xacro:macro name="wheel" params="prefix side x_pos y_pos friction">
     <link name="${prefix}_${side}_wheel">
       <visual>
         <geometry>
-          <cylinder radius="0.065" length="0.07"/> </geometry>
+          <cylinder radius="${wheel_radius}" length="${wheel_length}"/>
+        </geometry>
         <material name="black"/>
       </visual>
       <collision>
         <geometry>
-          <cylinder radius="0.065" length="0.07"/>
+          <cylinder radius="${wheel_radius}" length="${wheel_length}"/>
         </geometry>
       </collision>
@@ -57,10 +84,12 @@
     </gazebo>
   </xacro:macro>
-  <xacro:wheel prefix="mid" side="left"  x_pos="0"     y_pos="0.13" friction="1.0"/>
-  <xacro:wheel prefix="mid" side="right" x_pos="0"     y_pos="-0.13" friction="1.0"/>
-  <xacro:wheel prefix="front" side="left"  x_pos="0.16"  y_pos="0.13" friction="0.2"/>
-  <xacro:wheel prefix="front" side="right" x_pos="0.16"  y_pos="-0.13" friction="0.2"/>
-  <xacro:wheel prefix="rear" side="left"  x_pos="-0.16" y_pos="0.13" friction="0.2"/>
-  <xacro:wheel prefix="rear" side="right" x_pos="-0.16" y_pos="-0.13" friction="0.2"/>
+  <!-- WHEELS INSTANTIATION -->
+  <xacro:wheel prefix="mid" side="left"  x_pos="0" y_pos="${wheel_y_offset}" friction="1.0"/>
+  <xacro:wheel prefix="mid" side="right" x_pos="0" y_pos="-${wheel_y_offset}" friction="1.0"/>
+  <xacro:wheel prefix="front" side="left"  x_pos="${axle_x_offset}"  y_pos="${wheel_y_offset}" friction="0.2"/>
+  <xacro:wheel prefix="front" side="right" x_pos="${axle_x_offset}"  y_pos="-${wheel_y_offset}" friction="0.2"/>
+  <xacro:wheel prefix="rear" side="left"  x_pos="-${axle_x_offset}" y_pos="${wheel_y_offset}" friction="0.2"/>
+  <xacro:wheel prefix="rear" side="right" x_pos="-${axle_x_offset}" y_pos="-${wheel_y_offset}" friction="0.2"/>
+  <!-- LIDAR -->
   <link name="lidar_link">
     <visual>
@@ -83,6 +112,7 @@
     <parent link="base_link"/>
     <child link="lidar_link"/>
-    <origin xyz="0.05 0 0.10" rpy="0 0 0"/>
+    <origin xyz="${lidar_x} ${lidar_y} ${lidar_z}" rpy="0 0 ${lidar_yaw}"/>
   </joint>
+  <!-- IMU -->
   <link name="imu_link">
     <visual>
@@ -92,5 +122,5 @@
       <material name="green"/>
     </visual>
-        <collision>
+    <collision>
       <geometry>
         <cylinder radius="0.035" length="0.02"/>
@@ -105,12 +135,13 @@
     <parent link="base_link"/>
     <child link="imu_link"/>
-    <origin xyz="0.2 0 0.10" rpy="0 0 0"/>
-    </joint>
+    <origin xyz="${imu_x} ${imu_y} ${imu_z}" rpy="0 0 ${imu_yaw}"/>
+  </joint>
+  <!-- GAZEBO PLUGINS -->
   <gazebo>
     <plugin filename="gz-sim-diff-drive-system" name="gz::sim::systems::DiffDrive">
       <left_joint>mid_left_wheel_joint</left_joint>
       <right_joint>mid_right_wheel_joint</right_joint>
-      <wheel_separation>0.26</wheel_separation>
-      <wheel_radius>0.065</wheel_radius>
+      <wheel_separation>${wheel_y_offset * 2}</wheel_separation>
+      <wheel_radius>${wheel_radius}</wheel_radius>
       <topic>cmd_vel</topic>
       <max_linear_acceleration>2.0</max_linear_acceleration>
@@ -125,9 +156,11 @@
     </plugin>
     <plugin filename="gz-sim-joint-state-publisher-system" name="gz::sim::systems::JointStatePublisher">
-      <topic>joint_states</topic> <update_rate>30</update_rate>
+      <topic>joint_states</topic>
+      <update_rate>30</update_rate>
     </plugin>
     <plugin filename="gz-sim-imu-system" name="gz::sim::systems::Imu">
     </plugin>
   </gazebo>
+  <!-- GAZEBO SENSORS -->
   <gazebo reference="lidar_link">
     <sensor name="lidar" type="gpu_lidar">
@@ -162,40 +195,22 @@
         <angular_velocity>
           <x>
-            <noise type="gaussian">
-              <mean>0.0</mean>
-              <stddev>0.0</stddev>
-            </noise>
+            <noise type="gaussian"><mean>0.0</mean><stddev>0.0</stddev></noise>
           </x>
           <y>
-            <noise type="gaussian">
-              <mean>0.0</mean>
-              <stddev>0.0</stddev>
-            </noise>
+            <noise type="gaussian"><mean>0.0</mean><stddev>0.0</stddev></noise>
           </y>
           <z>
-            <noise type="gaussian">
-              <mean>0.0</mean>
-              <stddev>0.0</stddev>
-            </noise>
+            <noise type="gaussian"><mean>0.0</mean><stddev>0.0</stddev></noise>
           </z>
         </angular_velocity>
         <linear_acceleration>
           <x>
-            <noise type="gaussian">
-              <mean>0.0</mean>
-              <stddev>0.0</stddev>
-            </noise>
+            <noise type="gaussian"><mean>0.0</mean><stddev>0.0</stddev></noise>
           </x>
           <y>
-            <noise type="gaussian">
-              <mean>0.0</mean>
-              <stddev>0.0</stddev>
-            </noise>
+            <noise type="gaussian"><mean>0.0</mean><stddev>0.0</stddev></noise>
           </y>
           <z>
-            <noise type="gaussian">
-              <mean>0.0</mean>
-              <stddev>0.0</stddev>
-            </noise>
+            <noise type="gaussian"><mean>0.0</mean><stddev>0.0</stddev></noise>
           </z>
         </linear_acceleration>
@@ -203,5 +218,5 @@
       <topic>/imu</topic>
       <gz_frame_id>imu_link</gz_frame_id>
-      </sensor>
+    </sensor>
   </gazebo>
 </robot>

Commit message: working nav2 and slam with imu

File: src/hexarover_description/urdf/hexarover.urdf.xacro (robot description, xacro)
@@ -1,4 +1,26 @@
 <?xml version="1.0"?>
 <robot name="hexarover" xmlns:xacro="http://www.ros.org/wiki/xacro">
+  <!-- ================= WŁAŚCIWOŚCI (PROPERTIES) ================= -->
+  <!-- 1. WYMIARY GŁÓWNEJ BRYŁY (PODWOZIA) -->
+  <xacro:property name="chassis_length" value="0.38"/>
+  <xacro:property name="chassis_width"  value="0.12"/>
+  <xacro:property name="chassis_height" value="0.07"/>
+  <xacro:property name="chassis_z_offset" value="0.02"/>
+  <!-- 2. KOŁA -->
+  <xacro:property name="wheel_radius" value="0.0625"/>
+  <xacro:property name="wheel_length" value="0.06"/>
+  <xacro:property name="wheel_y_offset" value="0.12"/>
+  <xacro:property name="axle_x_offset" value="0.15"/>
+  <!-- 3. POZYCJA LIDARU -->
+  <xacro:property name="lidar_x" value="0.15"/>
+  <xacro:property name="lidar_y" value="0.00"/>
+  <xacro:property name="lidar_z" value="0.12"/>
+  <xacro:property name="lidar_yaw" value="0.0"/>
+  <!-- 4. POZYCJA IMU -->
+  <xacro:property name="imu_x" value="-0.15"/>
+  <xacro:property name="imu_y" value="0.00"/>
+  <xacro:property name="imu_z" value="0.06"/>
+  <xacro:property name="imu_yaw" value="0.0"/>
+  <!-- ========================================================== -->
   <material name="silver">
     <color rgba="0.8 0.8 0.8 1"/>
@@ -11,16 +33,19 @@
   </material>
   <material name="green">
-  <color rgba="0 1 0 1"/>
-  </material>
+    <color rgba="0 1 0 1"/>
+  </material>
+  <!-- BASE LINK -->
   <link name="base_link">
     <visual>
-      <origin xyz="0 0 0.04" rpy="0 0 0"/> <geometry>
-        <box size="0.45 0.16 0.08"/> </geometry>
+      <origin xyz="0 0 ${chassis_z_offset}" rpy="0 0 0"/>
+      <geometry>
+        <box size="${chassis_length} ${chassis_width} ${chassis_height}"/>
+      </geometry>
       <material name="silver"/>
     </visual>
     <collision>
-      <origin xyz="0 0 0.04" rpy="0 0 0"/>
-      <geometry>
-        <box size="0.45 0.16 0.08"/>
+      <origin xyz="0 0 ${chassis_z_offset}" rpy="0 0 0"/>
+      <geometry>
+        <box size="${chassis_length} ${chassis_width} ${chassis_height}"/>
       </geometry>
     </collision>
@@ -30,14 +55,16 @@
     </inertial>
   </link>
+  <!-- WHEEL MACRO -->
   <xacro:macro name="wheel" params="prefix side x_pos y_pos friction">
     <link name="${prefix}_${side}_wheel">
       <visual>
         <geometry>
-          <cylinder radius="0.065" length="0.07"/> </geometry>
+          <cylinder radius="${wheel_radius}" length="${wheel_length}"/>
+        </geometry>
         <material name="black"/>
       </visual>
       <collision>
         <geometry>
-          <cylinder radius="0.065" length="0.07"/>
+          <cylinder radius="${wheel_radius}" length="${wheel_length}"/>
         </geometry>
       </collision>
@@ -57,10 +84,12 @@
     </gazebo>
   </xacro:macro>
-  <xacro:wheel prefix="mid" side="left"  x_pos="0"     y_pos="0.13" friction="1.0"/>
-  <xacro:wheel prefix="mid" side="right" x_pos="0"     y_pos="-0.13" friction="1.0"/>
-  <xacro:wheel prefix="front" side="left"  x_pos="0.16"  y_pos="0.13" friction="0.2"/>
-  <xacro:wheel prefix="front" side="right" x_pos="0.16"  y_pos="-0.13" friction="0.2"/>
-  <xacro:wheel prefix="rear" side="left"  x_pos="-0.16" y_pos="0.13" friction="0.2"/>
-  <xacro:wheel prefix="rear" side="right" x_pos="-0.16" y_pos="-0.13" friction="0.2"/>
+  <!-- WHEELS INSTANTIATION -->
+  <xacro:wheel prefix="mid" side="left"  x_pos="0" y_pos="${wheel_y_offset}" friction="1.0"/>
+  <xacro:wheel prefix="mid" side="right" x_pos="0" y_pos="-${wheel_y_offset}" friction="1.0"/>
+  <xacro:wheel prefix="front" side="left"  x_pos="${axle_x_offset}"  y_pos="${wheel_y_offset}" friction="0.2"/>
+  <xacro:wheel prefix="front" side="right" x_pos="${axle_x_offset}"  y_pos="-${wheel_y_offset}" friction="0.2"/>
+  <xacro:wheel prefix="rear" side="left"  x_pos="-${axle_x_offset}" y_pos="${wheel_y_offset}" friction="0.2"/>
+  <xacro:wheel prefix="rear" side="right" x_pos="-${axle_x_offset}" y_pos="-${wheel_y_offset}" friction="0.2"/>
+  <!-- LIDAR -->
   <link name="lidar_link">
     <visual>
@@ -83,6 +112,7 @@
     <parent link="base_link"/>
     <child link="lidar_link"/>
-    <origin xyz="0.05 0 0.10" rpy="0 0 0"/>
+    <origin xyz="${lidar_x} ${lidar_y} ${lidar_z}" rpy="0 0 ${lidar_yaw}"/>
   </joint>
+  <!-- IMU -->
   <link name="imu_link">
     <visual>
@@ -92,5 +122,5 @@
       <material name="green"/>
     </visual>
-        <collision>
+    <collision>
       <geometry>
         <cylinder radius="0.035" length="0.02"/>
@@ -105,12 +135,13 @@
     <parent link="base_link"/>
     <child link="imu_link"/>
-    <origin xyz="0.2 0 0.10" rpy="0 0 0"/>
-    </joint>
+    <origin xyz="${imu_x} ${imu_y} ${imu_z}" rpy="0 0 ${imu_yaw}"/>
+  </joint>
+  <!-- GAZEBO PLUGINS -->
   <gazebo>
     <plugin filename="gz-sim-diff-drive-system" name="gz::sim::systems::DiffDrive">
       <left_joint>mid_left_wheel_joint</left_joint>
       <right_joint>mid_right_wheel_joint</right_joint>
-      <wheel_separation>0.26</wheel_separation>
-      <wheel_radius>0.065</wheel_radius>
+      <wheel_separation>${wheel_y_offset * 2}</wheel_separation>
+      <wheel_radius>${wheel_radius}</wheel_radius>
       <topic>cmd_vel</topic>
       <max_linear_acceleration>2.0</max_linear_acceleration>
@@ -125,9 +156,11 @@
     </plugin>
     <plugin filename="gz-sim-joint-state-publisher-system" name="gz::sim::systems::JointStatePublisher">
-      <topic>joint_states</topic> <update_rate>30</update_rate>
+      <topic>joint_states</topic>
+      <update_rate>30</update_rate>
     </plugin>
     <plugin filename="gz-sim-imu-system" name="gz::sim::systems::Imu">
     </plugin>
   </gazebo>
+  <!-- GAZEBO SENSORS -->
   <gazebo reference="lidar_link">
     <sensor name="lidar" type="gpu_lidar">
@@ -135,5 +168,5 @@
       <always_on>true</always_on>
       <visualize>true</visualize>
-      <update_rate>10</update_rate>
+      <update_rate>5</update_rate>
       <ray>
         <scan>
@@ -158,44 +191,26 @@
       <always_on>true</always_on>
       <visualize>true</visualize>
-      <update_rate>10</update_rate>
+      <update_rate>5</update_rate>
       <imu>
         <angular_velocity>
           <x>
-            <noise type="gaussian">
-              <mean>0.0</mean>
-              <stddev>0.0</stddev>
-            </noise>
+            <noise type="gaussian"><mean>0.0</mean><stddev>0.0</stddev></noise>
           </x>
           <y>
-            <noise type="gaussian">
-              <mean>0.0</mean>
-              <stddev>0.0</stddev>
-            </noise>
+            <noise type="gaussian"><mean>0.0</mean><stddev>0.0</stddev></noise>
           </y>
           <z>
-            <noise type="gaussian">
-              <mean>0.0</mean>
-              <stddev>0.0</stddev>
-            </noise>
+            <noise type="gaussian"><mean>0.0</mean><stddev>0.0</stddev></noise>
           </z>
         </angular_velocity>
         <linear_acceleration>
           <x>
-            <noise type="gaussian">
-              <mean>0.0</mean>
-              <stddev>0.0</stddev>
-            </noise>
+            <noise type="gaussian"><mean>0.0</mean><stddev>0.0</stddev></noise>
           </x>
           <y>
-            <noise type="gaussian">
-              <mean>0.0</mean>
-              <stddev>0.0</stddev>
-            </noise>
+            <noise type="gaussian"><mean>0.0</mean><stddev>0.0</stddev></noise>
           </y>
           <z>
-            <noise type="gaussian">
-              <mean>0.0</mean>
-              <stddev>0.0</stddev>
-            </noise>
+            <noise type="gaussian"><mean>0.0</mean><stddev>0.0</stddev></noise>
           </z>
         </linear_acceleration>
@@ -203,5 +218,5 @@
       <topic>/imu</topic>
       <gz_frame_id>imu_link</gz_frame_id>
-      </sensor>
+    </sensor>
   </gazebo>
 </robot>

Commit message: Added camera, human, yolo without human tracking

File: src/hexarover_description/urdf/hexarover.urdf.xacro (robot description, xacro)
@@ -137,4 +137,18 @@
     <origin xyz="${imu_x} ${imu_y} ${imu_z}" rpy="0 0 ${imu_yaw}"/>
   </joint>
+  <!-- CAMERA -->
+  <link name="camera_link">
+  <visual>
+    <geometry>
+      <box size="0.02 0.05 0.03"/>
+    </geometry>
+    <material name="black"/>
+  </visual>
+</link>
+<joint name="camera_joint" type="fixed">
+  <parent link="base_link"/>
+  <child link="camera_link"/>
+  <origin xyz="0.2 0 0.05" rpy="0 0 0"/>
+</joint>
   <!-- GAZEBO PLUGINS -->
   <gazebo>
@@ -220,3 +234,22 @@
     </sensor>
   </gazebo>
+  <gazebo reference="camera_link">
+  <sensor name="camera" type="camera">
+    <camera>
+      <horizontal_fov>1.34</horizontal_fov> <image>
+        <width>800</width>
+        <height>600</height>
+        <format>R8G8B8</format>
+      </image>
+      <clip>
+        <near>0.1</near>
+        <far>10.0</far>
+      </clip>
+    </camera>
+    <always_on>1</always_on>
+    <update_rate>30</update_rate>
+    <visualize>true</visualize>
+    <topic>image_raw</topic>
+  </sensor>
+</gazebo>
 </robot>
